Commit message: fix(s2b-a8): correct the FR3's mass properties (ruling 10); Panda finger fixes
- ROBOTS[robot]["mass_override"] maps each USD link to a franka_description link to
  copy or to (mass, com, inertia); "fer" stays the Panda's whole-arm shorthand. FR3:
  fr3_link8 and fr3_hand_tcp (1.0 kg bodies in Isaac 6.0's asset) become 1 g with a
  1e-7 inertia; fr3_hand and both fingers take franka_description's; link0..7 keep
  the asset's. The layer is committed as robots/fr3/fr3.usda, and description.json
  records the asset's PhysX masses next to the override's.
- franka_description's right finger frame is the USD's turned pi about z (both
  assets; checked for the Panda against fer.urdf.xacro): its COM and inertia are
  re-expressed, so the Panda's right finger no longer sits on the left one's side.
- A mimic joint takes its leader's velocity (panda_finger_joint2 had 10.0 m/s).
- pipeline_version 2. Reruns: FR3 4.5 %, M 1.0e-6, g 3.0e-6; Panda 6.4 %, M 3.5e-6,
  g 6.3e-6; all checks pass.

File: guide_motion/guide_motion/robots/fr3/fr3.urdf (robot description, URDF)
Before this commit: robot fr3, 13 links, 12 joints
Links:
- link fr3_hand: mass 0.7300000191 -> 0.654399991
- link fr3_hand_tcp: mass 1 -> 0.001000000047
- link fr3_leftfinger: mass 0.01513542887 -> 0.029099999
- link fr3_link8: mass 1 -> 0.001000000047
- link fr3_rightfinger: mass 0.01513542887 -> 0.029099999

File: guide_motion/guide_motion/robots/panda/panda.urdf (robot description, URDF)
Before this commit: robot panda, 12 links, 11 joints
Joints:
- joint panda_finger_joint2: limit lower=0 upper=0.04 effort=7.199999809 velocity=10.00000028 -> lower=0 upper=0.04 effort=7.199999809 velocity=0.2000000857
