Commit message: fix(s2b-final): the Panda's tool frame goes along the USD hand's z, not the exporter link's
C1: fix_urdf added panda_hand_tcp at 0 0 0.1034 in the exporter's hand link, which
is the USD (franka_description) hand turned 90 deg, so the TCP sat 10.3 cm beside
the hand with its z horizontal. build() now adds a missing TCP through
set_inertials' extra_links at frames[hand] @ T_z(0.1034). Panda home TCP
[0.3069, 0, 0.4869], z down: 0.0009 mm / 0.0001 deg from the FR3's (new Kit-free
test). The TCP test now uses a rotated hand frame. Regenerated with the Kit CLI:
only the TCP joint changed; checks unchanged (6.4 %, M 3.5e-6, g 6.3e-6); panda.xrdf
and all FR3 outputs byte-identical.
Parked 27: the one-entry _FD_TO_USD dict is an endswith("rightfinger") check.

File: guide_motion/guide_motion/robots/panda/panda.urdf (robot description, URDF)
Before this commit: robot panda, 12 links, 11 joints
Joints:
- removed joint panda_hand_tcp_joint
- added joint panda_hand_tcp_fixed: type fixed, parent panda_hand, child panda_hand_tcp, origin xyz=-0.1034002325 -1.167997758e-07 -3.308135054e-08 rpy=1.570796409 -0.785397933 -1.570796368
